Commit message: Update robot.urdf
update of robot for small one

File: catkin_ws/src/burf_robot/robot.urdf (robot description, URDF)
Before this commit: robot robot_model, 5 links, 4 joints
Links:
- link base_frame: geometry collision box size=0.35 0.35 0.15; visual box size=0.30 0.30 0.15
Joints:
- joint base_to_lwheel: origin xyz=0 0.42 0.06 rpy=1.5708 0 0 -> xyz=0 0.17 0.06 rpy=1.5708 0 0
- joint base_to_rwheel: origin xyz=0 -0.42 0.06 rpy=-1.5708 0 0 -> xyz=0 -0.17 0.06 rpy=-1.5708 0 0
- joint laser_joint: origin xyz=-0.5 0.0 0.80 rpy=0 0 0 -> xyz=0.15 0.0 0.30 rpy=0 0 0
